File: Schema/Proto-1/Proto-1.kicad_sch (KiCad schematic)
At the start: 5 parts, among them J1 Conn_02x03_Top_Bottom, U1 ATtiny85V-10P

Commit message: Benenne Files um
Parts:
- J1: value Conn_02x03_Top_Bottom -> Conn_02x03
Changed lines of the file:
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@@
 			)
 		)
-		(property "Value" "Conn_02x03_Top_Bottom"
+		(property "Value" "Conn_02x03"
 			(at 93.98 69.85 0)
 			(effects

Commit message: Erstelle Schema für B
Connections:
- net Reset: now reaches J1.4 (Pin_4)
- net Reset: now also U1.1 (~{RESET}/PB5)
- no-connect marks 4 -> 2
Other:
- added sheet Proto-1b (Proto-1b.kicad_sch)
Changed lines of the file:
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@@
 		(at 74.93 53.34)
 	)
-	(no_connect
-		(at 100.33 73.66)
-	)
-	(no_connect
-		(at 74.93 55.88)
+	(wire
+		(pts
+			(xy 74.93 55.88) (xy 80.01 55.88)
+		)
+		(stroke
+			(width 0)
+			(type default)
+		)
 	)
 	(wire
@@
 	(wire
 		(pts
+			(xy 102.87 73.66) (xy 100.33 73.66)
+		)
+		(stroke
+			(width 0)
+			(type default)
+		)
+	)
+	(wire
+		(pts
 			(xy 105.41 78.74) (xy 109.22 78.74)
 		)
@@
 	(wire
 		(pts
+			(xy 102.87 69.85) (xy 102.87 73.66)
+		)
+		(stroke
+			(width 0)
+			(type default)
+		)
+	)
+	(wire
+		(pts
+			(xy 105.41 69.85) (xy 102.87 69.85)
+		)
+		(stroke
+			(width 0)
+			(type default)
+		)
+	)
+	(wire
+		(pts
 			(xy 59.69 66.04) (xy 59.69 68.58)
 		)
@@
 			(width 0)
 			(type default)
+		)
+	)
+	(global_label "Reset"
+		(shape input)
+		(at 105.41 69.85 0)
+		(fields_autoplaced yes)
+		(effects
+			(font
+				(size 1.27 1.27)
+			)
+			(justify left)
+		)
+		(property "Intersheetrefs" "${INTERSHEET_REFS}"
+			(at 113.5962 69.85 0)
+			(effects
+				(font
+					(size 1.27 1.27)
+				)
+				(justify left)
+				(hide yes)
+			)
 		)
 	)
@@
 				)
 				(justify right)
+				(hide yes)
+			)
+		)
+	)
+	(global_label "Reset"
+		(shape input)
+		(at 80.01 55.88 0)
+		(fields_autoplaced yes)
+		(effects
+			(font
+				(size 1.27 1.27)
+			)
+			(justify left)
+		)
+		(property "Intersheetrefs" "${INTERSHEET_REFS}"
+			(at 88.1962 55.88 0)
+			(effects
+				(font
+					(size 1.27 1.27)
+				)
+				(justify left)
 				(hide yes)
 			)
@@
 				)
 			)
+		)
+	)
+	(sheet
+		(at 336.55 -21.59)
+		(size 213.36 125.73)
+		(exclude_from_sim no)
+		(in_bom yes)
+		(on_board yes)
+		(dnp no)
+		(fields_autoplaced yes)
+		(stroke
+			(width 0.1524)
+			(type solid)
+		)
+		(fill
+			(color 0 0 0 0.0000)
+		)
+		(property "Sheetname" "Proto-1b"
+			(at 336.55 -22.3016 0)
+			(effects
+				(font
+					(size 1.27 1.27)
+				)
+				(justify left bottom)
+			)
+		)
+		(property "Sheetfile" "Proto-1b.kicad_sch"
+			(at 336.55 104.7246 0)
+			(effects
+				(font
+					(size 1.27 1.27)
+				)
+				(justify left top)
+			)
+		)
+		(instances
+			(project "Proto-1"
+				(path "/ad20f11c-8bda-436c-a37e-51accbad252d"
+					(page "2")
+				)
+			)

Commit message: Beginne Devboard
Parts:
- removed D1, D2, D3: WS2812B, LED_SMD:LED_WS2812B_PLCC4_5.0x5.0mm_P3.2mm, symbol LED:WS2812B
- removed J1: Conn_02x03, Connector_IDC:IDC-Header_2x03_P2.54mm_Horizontal, symbol Connector_Generic:Conn_02x03_Top_Bottom
- removed U1: ATtiny85V-10P, Package_SO:SO-8_3.9x4.9mm_P1.27mm, symbol MCU_Microchip_ATtiny:ATtiny85V-10P
Connections:
- no-connect marks 2 -> 0
Other:
- added sheet DevBoard esp32c6 (devboard-esp32c6.kicad_sch)
- added sheet Proto-1a (proto-1a.kicad_sch)
