File: Schema/Proto-1/devboard-esp32c6.kicad_sch (KiCad schematic)
At the start: 8 parts, among them J3 Conn_02x02_Counter_Clockwise, U2 ESP32-DevKitM-1

Commit message: Erstelle PCB für Devboard, ersetzte Proto-1-Board
Connections:
- net +5V: now also J3.3 (Pin_3); no longer J3.1 (Pin_1)
- net at D10.4 (DIN): now also J3.1 (Pin_1); no longer J3.3 (Pin_3)
Changed lines of the file:
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@@
-	(wire
-		(pts
-			(xy 132.08 82.55) (xy 144.78 82.55)
-		)
-		(stroke
-			(width 0)
-			(type default)
-		)
-	)
-	(wire
-		(pts
-			(xy 111.76 45.72) (xy 111.76 55.88)
-		)
-		(stroke
-			(width 0)
-			(type default)
-		)
-	)
 	(wire
 		(pts
@@
 	(wire
 		(pts
-			(xy 128.27 58.42) (xy 132.08 58.42)
-		)
-		(stroke
-			(width 0)
-			(type default)
-		)
-	)
-	(wire
-		(pts
 			(xy 72.39 19.05) (xy 72.39 30.48)
 		)
@@
 	(wire
 		(pts
-			(xy 132.08 58.42) (xy 132.08 82.55)
-		)
-		(stroke
-			(width 0)
-			(type default)
-		)
-	)
-	(wire
-		(pts
 			(xy 171.45 72.39) (xy 170.18 72.39)
 		)
@@
 	(wire
 		(pts
+			(xy 128.27 58.42) (xy 128.27 63.5)
+		)
+		(stroke
+			(width 0)
+			(type default)
+		)
+	)
+	(wire
+		(pts
 			(xy 156.21 40.64) (xy 167.64 40.64)
 		)
@@
 	(wire
 		(pts
-			(xy 115.57 58.42) (xy 111.76 58.42)
+			(xy 128.27 63.5) (xy 132.08 63.5)
 		)
 		(stroke
@@
 	(wire
 		(pts
-			(xy 111.76 58.42) (xy 111.76 64.77)
-		)
-		(stroke
-			(width 0)
-			(type default)
-		)
-	)
-	(wire
-		(pts
 			(xy 154.94 57.15) (xy 154.94 77.47)
 		)
@@
 	(wire
 		(pts
+			(xy 111.76 82.55) (xy 111.76 55.88)
+		)
+		(stroke
+			(width 0)
+			(type default)
+		)
+	)
+	(wire
+		(pts
 			(xy 132.08 40.64) (xy 140.97 40.64)
 		)
@@
 		(pts
 			(xy 175.26 52.07) (xy 200.66 52.07)
+		)
+		(stroke
+			(width 0)
+			(type default)
+		)
+	)
+	(wire
+		(pts
+			(xy 111.76 82.55) (xy 144.78 82.55)
 		)
 		(stroke
@@
 	(symbol
 		(lib_id "power:+5V")
-		(at 111.76 45.72 0)
+		(at 132.08 63.5 0)
 		(unit 1)
 		(exclude_from_sim no)
@@
 		(fields_autoplaced yes)
 		(property "Reference" "#PWR017"
-			(at 111.76 49.53 0)
+			(at 132.08 67.31 0)
 			(effects
 				(font
@@
 		)
 		(property "Value" "+5V"
-			(at 111.76 40.64 0)
+			(at 132.08 58.42 0)
 			(effects
 				(font
@@
 		)
 		(property "Footprint" ""
-			(at 111.76 45.72 0)
+			(at 132.08 63.5 0)
 			(effects
 				(font
@@
 		)
 		(property "Datasheet" ""
-			(at 111.76 45.72 0)
+			(at 132.08 63.5 0)
 			(effects
 				(font
@@
 		)
 		(property "Description" "Power symbol creates a global label with name \"+5V\""
-			(at 111.76 45.72 0)
+			(at 132.08 63.5 0)
 			(effects
 				(font
@@
 		(exclude_from_sim no)
 		(in_bom yes)
-		(on_board yes)
+		(on_board no)
 		(dnp no)
 		(fields_autoplaced yes)
@@
 	(symbol
 		(lib_id "power:GND")
-		(at 111.76 64.77 0)
+		(at 115.57 58.42 0)
 		(unit 1)
 		(exclude_from_sim no)
@@
 		(fields_autoplaced yes)
 		(property "Reference" "#PWR018"
-			(at 111.76 71.12 0)
+			(at 115.57 64.77 0)
 			(effects
 				(font
@@
 		)
 		(property "Value" "GND"
-			(at 111.76 69.85 0)
+			(at 115.57 63.5 0)
 			(effects
 				(font
@@
 		)
 		(property "Footprint" ""
-			(at 111.76 64.77 0)
+			(at 115.57 58.42 0)
 			(effects
 				(font
@@
 		)
 		(property "Datasheet" ""
-			(at 111.76 64.77 0)
+			(at 115.57 58.42 0)
 			(effects
 				(font
@@
 		)
 		(property "Description" "Power symbol creates a global label with name \"GND\" , ground"
-			(at 111.76 64.77 0)
-			(effects
-				(font
+			(at 115.57 58.42 0)
+			(effects
+				(font

Commit message: Bereite DB1-0.4 vor
Other:
- note added: "${Version}"
- note added: "Development Board ESP32-C6"
Changed lines of the file:
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@@
 	(generator_version "9.0")
 	(paper "A4")
+	(text "${Version}"
+		(exclude_from_sim no)
+		(at 274.066 193.294 0)
+		(effects
+			(font
+				(size 1.27 1.27)
+			)
+		)
+	)
+	(text "Development Board ESP32-C6"
+		(exclude_from_sim no)
+		(at 207.772 189.992 0)
+		(effects
+			(font
+				(size 1.778 1.778)
+				(thickness 0.3556)
+				(bold yes)
+			)
+		)
+	)
 	(junction
 		(at 148.59 26.67)

Commit message: Bereite Proto-1-0.5a vor, setze Sheet-Propery "exclude from board"
Parts:
- D4, D8: Component Class (none) -> DevBoard
Changed lines of the file:
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@@
+			)
+		)
+		(property "Component Class" "DevBoard"
+			(at 148.59 40.64 0)
+			(effects
+				(font
+					(size 1.27 1.27)
+				)
+				(hide yes)
 			)
 		)
@@
 			(at 175.26 40.64 0)
 			(effects
+				(font
+					(size 1.27 1.27)
+				)
+				(hide yes)
+			)
+		)
+		(property "Component Class" "DevBoard"
+			(at 175.26 40.64 0)
+			(effects
