File: Schema/rpi-zero-platine/rpi-zero-platine.kicad_sch (KiCad schematic)
At the start: 4 parts, among them J1 GPIO, J2 Screw_Terminal_01x06, J3 Screw_Terminal_01x02, SW1 SW_DIP_x02

Commit message: Überarbeite Platine
Parts:
- added J1: GPIO, Connector_PinSocket_2.54mm:PinSocket_2x13_P2.54mm_Vertical, symbol Connector_Generic:Conn_02x13_Odd_Even
- J2: footprint TerminalBlock_Altech:Altech_AK100_1x06_P5.00mm -> TerminalBlock_Phoenix:TerminalBlock_Phoenix_MKDS-1,5-6-5.08_1x06_P5.08mm_Horizontal
- J3: footprint TerminalBlock:TerminalBlock_Altech_AK300-2_P5.00mm -> TerminalBlock_Phoenix:TerminalBlock_Phoenix_MKDS-1,5-2-5.08_1x02_P5.08mm_Horizontal
- J7: renamed from J1; value GPIO -> GPIO-alt
- SW1: footprint Button_Switch_THT:SW_DIP_SPSTx02_Piano_10.8x6.64mm_W7.62mm_P2.54mm -> Button_Switch_THT:SW_PUSH_6mm_H4.3mm; symbol Switch:SW_DIP_x02 -> Switch:SW_DIP_x01
Connections:
- net +5V: now also J3.2 (Pin_2), J1.2 (VCC); no longer J3.1 (Pin_1), J7.2 (Pin_2), J7.4 (Pin_4)
- net GND: now also J3.1 (Pin_1), J1.25 (GND); no longer J3.2 (Pin_2), J7.14 (Pin_14), J7.20 (Pin_20), J7.25 (Pin_25), J7.30 (Pin_30), J7.34 (Pin_34), J7.39 (Pin_39), J7.6 (Pin_6), J7.9 (Pin_9), SW1.4
- net GPIO10/SPI0.MOSI: no longer J2.4 (Pin_4)
- net GPIO11/SPI0.SCLK: no longer J2.5 (Pin_5)
- net at SW1.2: now also J1.15 (Pin_15)
- net +3V3: no longer names the net of J7.1 (Pin_1)
- net +3V3: no longer J7.17 (Pin_17)
- net GPIO17: no longer names the net of J7.11 (Pin_11)
- net GPIO17: no longer SW1.1
- new net: J7.25 (Pin_25), J7.39 (Pin_39), J7.9 (Pin_9)
- new net: J1.19 (SPI0.MOSI), J2.5 (Pin_5)
- new net: J1.23 (SPI0.SCLK), J2.4 (Pin_4)
- new net: J1.9 (Pin_9), SW1.1
- no-connect marks 27 -> 57
Other:
- moved on the sheet: J2, J3

Commit message: Beschriftung
Parts:
- J2: value Screw_Terminal_01x06 -> LED Out A
- J3: value Screw_Terminal_01x02 -> LED Out B
Connections:
- net Data: now reaches J1.19 (SPI0.MOSI), J2.5 (Pin_5)
- net Clock: now reaches J1.23 (SPI0.SCLK), J2.4 (Pin_4)
Changed lines of the file:
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@@
 	(text_box "Kabelfarben\n- Clock gelb\n- Data blau"
 		(exclude_from_sim no)
-		(at 227.33 26.67 0)
+		(at 207.01 26.67 0)
 		(size 24.13 21.59)
 		(margins 0.9525 0.9525 0.9525 0.9525)
@@
 		)
 	)
+	(label "Clock"
+		(at 162.56 72.39 0)
+		(effects
+			(font
+				(size 1.27 1.27)
+			)
+			(justify left bottom)
+		)
+	)
 	(label "GPIO2{slash}SDA1"
 		(at 31.75 30.48 0)
@@
 			)
 			(justify right bottom)
+		)
+	)
+	(label "Data"
+		(at 162.56 74.93 0)
+		(effects
+			(font
+				(size 1.27 1.27)
+			)
+			(justify left bottom)
 		)
 	)
@@
 		(on_board yes)
 		(dnp no)
-		(fields_autoplaced yes)
 		(property "Reference" "J2"
-			(at 194.31 39.3699 0)
+			(at 191.77 32.004 0)
 			(effects
 				(font
@@
 			)
 		)
-		(property "Value" "Screw_Terminal_01x06"
-			(at 194.31 41.9099 0)
+		(property "Value" "LED Out A"
+			(at 194.818 46.482 90)
 			(effects
 				(font
@@
 		(on_board yes)
 		(dnp no)
-		(fields_autoplaced yes)
 		(property "Reference" "J3"
-			(at 194.31 54.6099 0)
+			(at 191.008 52.07 0)
 			(effects
 				(font
@@
 			)
 		)
-		(property "Value" "Screw_Terminal_01x02"
-			(at 194.31 57.1499 0)
-			(effects
-				(font
+		(property "Value" "LED Out B"
+			(at 194.564 60.198 90)
+			(effects
+				(font
